File: EDA/esp32-r7-data-logger/esp32-r7-data-logger.kicad_sch (KiCad schematic)
At the start: 8 parts, among them J1 Conn_01x02, U1 ESP32-WROOM-32U

Commit message: Updates to EDA files for symbols that don't throw errors during ERC
Parts:
- removed C1: 22uF, easyeda2kicad:C1206, symbol LCSC:CL31B226KPHNNNE
- removed C2: 10uF, easyeda2kicad:C1206, symbol LCSC:CL31B104KBCNNNC
- removed J1: Conn_01x02, symbol Connector_Generic:Conn_01x02
- removed R1: 1206W4F3301T5E, easyeda2kicad:R1206, symbol LCSC:1206W4F3301T5E
- removed R3: 10k, easyeda2kicad:R1206, symbol LCSC:1206W4F1002T5E
- removed U1: ESP32-WROOM-32U, easyeda2kicad:WIFIM-SMD_38P-L19.2-W18.0-P1.27, symbol LCSC:ESP32-WROOM-32U
- added C1, C3, C5: 10uF, easyeda2kicad:C1206, symbol Device:C
- added C2, C4, C7: 22uF, easyeda2kicad:C1206, symbol Device:C
- added CN1: ZX-XH2.54-2PWT, easyeda2kicad:CONN-SMD_2P-P2.54_MEGASTAR_ZX-XH2.54-2PWT, symbol LCSC:ZX-XH2.54-2PWT
- added H1, H2, H3, H4: MountingHole, MountingHole:MountingHole_2.5mm, symbol Mechanical:MountingHole
- added L2: 3.9uH, easyeda2kicad:L1210, symbol Device:L_Small
- added R1, R3: 10k, easyeda2kicad:R1206, symbol Device:R
- added U2, U7: ZX-XH2.54-4PWT, easyeda2kicad:CONN-SMD_4P-P2.50-WAFER-254W-4P, symbol LCSC:ZX-XH2.54-4PWT
- added U3: AP63203WU-7, easyeda2kicad:TSOT-26_L2.9-W1.6-P0.95-LS2.8-BL, symbol LCSC:AP63203WU-7
- added U4: ESP32-WROOM-32UE, easyeda2kicad:WIFIM-SMD_38P-L19.2-W18.0-P1.27, symbol RF_Module:ESP32-WROOM-32UE
- added U5: ZX-XH2.54-6PWT, easyeda2kicad:CONN-SMD_ZX-XH2.54-6PWT, symbol LCSC:ZX-XH2.54-6PWT
- added U6: SN65HVD230DR, easyeda2kicad:SOIC-8_L4.9-W3.9-P1.27-LS6.0-BL, symbol LCSC:SN65HVD230DR
Connections:
- net +3.3V: now also C2.1, C3.1, C4.1, C7.1, L2.2, R1.1, U2.1, U3.1 (FB), U4.2 (VDD), U5.5, U6.3 (VCC); no longer Card1.7 (DAT0)
- net CLK: now also U4.13 (IO14)
- net CMD: now also U4.23 (IO15)
- net D1: now also U4.26 (IO4)
- net D2: now also U4.14 (IO12)
- net D3: now also U4.16 (IO13)
- net GND: now also C2.2, C3.2, C4.2, C5.2, C7.2, CN1.2, R3.2, U2.2, U3.4 (GND), U4.1 (GND), U4.15 (GND), U4.38 (GND), U4.39 (GND), U5.6, U6.2 (GND), U7.2
- net D0: now reaches R2.1
- net D0: now also Card1.7 (DAT0), CN1.1, U4.24 (IO2)
- new net: C1.2, L2.1, U3.5 (SW)
- new net: C1.1, U3.6 (BST)
- new net +12V: C5.1, U3.2 (EN), U3.3 (VIN), U7.1
- new net CANH: U6.7 (CANH), U7.3
- new net CANL: U6.6 (CANL), U7.4
- new net CAN_RS: R3.1, U6.8 (RS)
- new net CAN_RX: U4.27 (IO16), U6.4 (R)
- new net CAN_TX: U4.28 (IO17), U6.1 (D)
- new net EN: R1.2, U4.3 (EN), U5.4
- new net ESP32_RX: U4.34 (RXD0/IO3), U5.2
- new net ESP32_TX: U4.35 (TXD0/IO1), U5.1
- new net I2C_SCL: U2.4, U4.36 (IO22)
- new net I2C_SDA: U2.3, U4.33 (IO21)
- new net IO0: U4.25 (IO0), U5.3
- no-connect marks 0 -> 28
Other:
- note added: "CAN Communication"
- note added: "Fast SD Card"
- note added: "GPS"
- note added: "MCU & Programming"
- note added: "Power Converter"
- moved on the sheet: Card1, R2
